File: Boards/Carte_PAMI/Carte_PAMI.kicad_pcb (KiCad board)
At the start: 4 copper layers, 80 x 62 mm, 41 parts, among them J1 Emergency BTN, J10 DC Motor B, J2 USB_C_Receptacle_USB2.0_16P, J3 VL53L0X_1, J4 VL53L0X_2, J5 Battery_connector, J6 ELRS_Module, J7 Tirette, J8 DC Motor A, J9 Odom_Shield, Q1 PMOS, SW1 SW_Push, SW2 SW_Push, SW3 SW_Nidec_CAS-120A1, U1 ESP32-S3-WROOM-1U-N16R8, U2 USBLC6-2SC6, U3 TLV76150DCY, U4 TLV76133DCY, U5 TB6612FNG

Commit message: V1.1 : first layout
Parts:
- removed D1: B120-E3, Diode_SMD:D_SMA
- removed R9: 10k, Resistor_SMD:R_1206_3216Metric
- added C11: 22uF, Capacitor_SMD:C_0805_2012Metric, F.Cu at (102.1, 66.0)
- added C12: 22uF, Capacitor_SMD:C_0805_2012Metric, F.Cu at (104.8, 66.0)
- added C13: 1uF, Capacitor_SMD:C_0805_2012Metric, F.Cu at (105.5, 60.5)
- added C14: 2.2uF, Capacitor_SMD:C_0805_2012Metric, F.Cu at (113.8, 52.2)
- added D4: PWRLED, LED_SMD:LED_1206_3216Metric, F.Cu at (85.4, 72.1)
- added H1: MountingHole, MountingHole:MountingHole_2.2mm_M2, F.Cu at (70.0, 45.0)
- added H2: MountingHole, MountingHole:MountingHole_2.2mm_M2, F.Cu at (165.0, 45.0)
- added H3: MountingHole, MountingHole:MountingHole_2.2mm_M2, F.Cu at (192.8, 114.6)
- added H4: MountingHole, MountingHole:MountingHole_2.2mm_M2, F.Cu at (165.0, 115.0)
- added J11: Conn_01x08_Pin, Connector_PinHeader_2.54mm:PinHeader_1x08_P2.54mm_Vertical, F.Cu at (137.5, 52.0)
- added J12: JTAG interface, Connector_PinHeader_2.54mm:PinHeader_1x04_P2.54mm_Vertical, F.Cu at (150.5, 77.5)
- added L1: 3.3uH, Inductor_SMD:L_0805_2012Metric, F.Cu at (99.5, 65.9)
- added R10: 300, Resistor_SMD:R_1206_3216Metric, F.Cu at (89.6, 70.7)
- added SW4: SW_Nidec_CAS-120A1, Button_Switch_SMD:Nidec_Copal_CAS-120A, F.Cu at (140.4, 82.0)
- C1: value 22uF -> 10uF; footprint Capacitor_SMD:C_1206_3216Metric -> Capacitor_SMD:C_0805_2012Metric
- C10: value 2.2uF -> 0.1uF
- C2: value 0.1uF -> 22uF; footprint Capacitor_SMD:C_0805_2012Metric -> Capacitor_SMD:C_1206_3216Metric
- C5: value 1uF -> 10uF
- C6: value 10uF -> 0.1uF; footprint Capacitor_SMD:C_1206_3216Metric -> Capacitor_SMD:C_0805_2012Metric
- C7: value 0.1uF -> 10uF
- C8: value 1uF -> 0.1uF; footprint Capacitor_SMD:C_0805_2012Metric -> Capacitor_SMD:C_1206_3216Metric
- C9: value 2.2uF -> 1uF
- D3: value PWRLED -> B120-E3; footprint LED_SMD:LED_1206_3216Metric -> Diode_SMD:D_SMA
- J1: value Emergency BTN -> Battery_connector
- J10: value DC Motor B -> Battery_connector; footprint Connector_PinHeader_2.54mm:PinHeader_1x02_P2.54mm_Vertical -> Connector_JST:JST_XH_B2B-XH-A_1x02_P2.50mm_Vertical
- J5: value Battery_connector -> Tirette
- J7: value Tirette -> DC Motor B; footprint Connector_JST:JST_XH_B2B-XH-A_1x02_P2.50mm_Vertical -> Connector_PinHeader_2.54mm:PinHeader_1x06_P2.54mm_Vertical
- J8: footprint Connector_PinHeader_2.54mm:PinHeader_1x02_P2.54mm_Vertical -> Connector_PinHeader_2.54mm:PinHeader_1x06_P2.54mm_Vertical
- R2: value 10k -> 16.2k
- R3: value 10k -> 5k1
- R4: value 16.2k -> 5k1
- R6: value 1k -> 10k
- R7: value 10k -> 54k9
- SW1: value SW_Push -> SW_Nidec_CAS-120A1; footprint Button_Switch_SMD:SW_SPST_PTS810 -> Button_Switch_SMD:Nidec_Copal_CAS-120A
- SW3: value SW_Nidec_CAS-120A1 -> SW_Push; footprint Button_Switch_SMD:Nidec_Copal_CAS-120A -> Button_Switch_SMD:SW_SPST_PTS810
- U1: value ESP32-S3-WROOM-1U-N16R8 -> TPS563201; footprint ESP32-S3-WROOM-1U:ESP32-S3-WROOM-1U_EXP -> Package_TO_SOT_SMD:SOT-23-6
- U3: value TLV76150DCY -> ESP32-S3-WROOM-1U-N16R8; footprint Package_TO_SOT_SMD:SOT-223-3_TabPin2 -> ESP32-S3-WROOM-1U:ESP32-S3-WROOM-1U_EXP
- moved J10 63.7 mm to (81.0, 64.8), turned to 90 degrees
- moved Q1 61.9 mm to (93.3, 55.1)
- moved J2 57.5 mm to (80.6, 81.7), turned to -90 degrees
- moved U2 50.3 mm to (90.4, 81.2)
- moved R8 47.0 mm to (88.2, 60.9), turned to 180 degrees
- moved SW1 46.4 mm to (88.3, 54.9)
- moved J1 45.1 mm to (81.0, 55.6), turned to 90 degrees
- moved C3 44.8 mm to (142.5, 100.5), turned to -90 degrees
- moved SW2 43.3 mm to (139.3, 99.4), turned to 90 degrees
- moved C1 40.6 mm to (98.9, 59.5)
- moved R7 39.7 mm to (89.7, 65.2), turned to -90 degrees
- moved C6 38.6 mm to (111.5, 65.7), turned to 90 degrees
- moved C8 37.5 mm to (89.0, 75.7), turned to -90 degrees
- moved J6 37.4 mm to (127.8, 58.0), turned to 90 degrees
- moved R5 35.5 mm to (93.9, 60.9)
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Connections:
- net Net-(J2-D+-PadA6) renamed USB_D+
- net Net-(J2-D--PadA7) renamed USB_D-
- C1 pad 1: +3.3V -> VBAT
- C10 pad 1: +3.3V -> Net-(U1-SW)
- C10 pad 2: GND -> Net-(U1-VBST)
- C2 pad 1: GND -> +3.3V
- C2 pad 2: EN -> GND
- C3 pad 2: BOOT -> EN
- C4 pad 1: +3.3V -> GND
- C4 pad 2: GND -> BOOT
- C5 pad 1: GND -> VBAT
- C5 pad 2: EN -> GND
- C6 pad 1: GND -> +3.3V
- C6 pad 2: VBUS -> GND
- C8 pad 1: VBUS -> GND
- C8 pad 2: GND -> VBUS
- C9 pad 1: +5V -> GND
- C9 pad 2: GND -> EN
- D2 pad 1: VBUS -> Net-(D2-K)
- D2 pad 2: VBAT -> VBUS
- D3 pad 1: GND -> Net-(D2-K)
- D3 pad 2: Net-(D3-A) -> +5V
- J10 pad 1: BO1 -> GND
- J10 pad 2: BO2 -> BAT_IN
- J2 pad A4: Net-(D1-A) -> VBUS
- J2 pad A9: Net-(D1-A) -> VBUS
- J2 pad B4: Net-(D1-A) -> VBUS
- J2 pad B9: Net-(D1-A) -> VBUS
- J3 pad 3: TOF_SDA_1 -> ODOM_SDA
- J3 pad 4: TOF_SCL_1 -> ODOM_SCL
- J4 pad 3: TOF_SDA_1 -> ODOM_SDA
- J4 pad 4: TOF_SCL_1 -> ODOM_SCL
- J5 pad 1: GND -> +3.3V
- J5 pad 2: BAT_IN -> TRIGGER
- J7 pad 1: +3.3V -> GND
- J7 pad 2: TRIGGER -> ENC_BO1
- J8 pad 1: AO1 -> GND
- J8 pad 2: AO2 -> ENC_AO1
- Q1 pad 1: Net-(J1-Pin_2) -> Net-(Q1-D)
- R1 pad 1: GND -> VBAT_SENSE
- R1 pad 2: Net-(J2-CC2) -> GND
- R2 pad 1: +3.3V -> VBAT_SENSE
- R2 pad 2: EN -> VBAT
- R3 pad 2: Net-(J2-CC1) -> Net-(J2-CC2)
- R4 pad 1: VBAT_SENSE -> GND
- R4 pad 2: VBAT -> Net-(J2-CC1)
- R5 pad 1: GND -> Net-(U1-EN)
- R5 pad 2: VBAT_SENSE -> VBAT
- R6 pad 1: Net-(D3-A) -> +3.3V
- R6 pad 2: VBUS -> EN
- R7 pad 1: +3.3V -> Net-(U1-VFB)
- R7 pad 2: TOF_INT_1 -> +5V
- R8 pad 1: +3.3V -> Net-(U1-VFB)
- R8 pad 2: TOF_INT_2 -> GND
- SW1 pad 1: GND -> Net-(J1-Pin_2)
- SW1 pad 2: EN -> Net-(Q1-D)
- SW2 pad 2: BOOT -> EN
- SW3 pad 2: Net-(SW3-B) -> BOOT
- U1 pad 2: +3.3V -> Net-(U1-SW)
- U1 pad 3: EN -> VBAT
- U1 pad 4: TOF_SHUT_1 -> Net-(U1-VFB)
- U1 pad 5: TOF_SHUT_2 -> Net-(U1-EN)
- U1 pad 6: TOF_INT_1 -> Net-(U1-VBST)
- U3 pad 2: Net-(U3-VO) -> +3.3V
- U3 pad 3: VBUS -> EN
- U4 pad 3: Net-(U3-VO) -> Net-(D2-K)
Routing:
- net VBAT: track 0.00 -> 81.4 mm
- net EN: track 0.00 -> 65.8 mm, vias 0 -> 2
- net +5V: track 0.00 -> 63.5 mm, vias 0 -> 1
- net GND: track 0.00 -> 61.1 mm, vias 0 -> 45
- net VBAT_SENSE: track 0.00 -> 37.6 mm, vias 0 -> 2
- net ENC_BO1: track 0.00 -> 36.2 mm, vias 0 -> 1
- net Net-(D2-K): track 0.00 -> 34.8 mm, vias 0 -> 4
- net ENC_BO2: track 0.00 -> 34.7 mm, vias 0 -> 1
- net IO8: track 0.00 -> 34.2 mm
- net IO18: track 0.00 -> 31.9 mm
- net ENC_AO1: track 0.00 -> 31.8 mm, vias 0 -> 1
- net ENC_AO2: track 0.00 -> 30.9 mm, vias 0 -> 1
- net IO17: track 0.00 -> 29.8 mm
- net IO16: track 0.00 -> 27.6 mm
- net TOF_INT_1: track 0.00 -> 25.9 mm, vias 0 -> 1
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Other:
- board size 80 x 62 mm -> 77 x 58 mm
