File: Boards/Carte_PAMI/Carte_PAMI.kicad_sch (KiCad schematic)
At the start: 1 part, among them U1 ESP32-S3-WROOM-1U-N16R8

Commit message: V1 of Schematic
Parts:
- added C1: 22uF, Capacitor_SMD:C_1206_3216Metric, symbol Device:C
- added C10, C9: 2.2uF, Capacitor_SMD:C_0805_2012Metric, symbol Device:C
- added C2, C3, C4: 0.1uF, Capacitor_SMD:C_0805_2012Metric, symbol Device:C
- added C5, C8: 1uF, Capacitor_SMD:C_0805_2012Metric, symbol Device:C
- added C6: 10uF, Capacitor_SMD:C_1206_3216Metric, symbol Device:C
- added C7: 0.1uF, Capacitor_SMD:C_1206_3216Metric, symbol Device:C
- added D1, D2: B120-E3, Diode_SMD:D_SMA, symbol Diode:B120-E3
- added D3: PWRLED, LED_SMD:LED_1206_3216Metric, symbol Device:LED
- added J1: Emergency BTN, Connector_JST:JST_XH_B2B-XH-A_1x02_P2.50mm_Vertical, symbol Connector_Generic:Conn_01x02
- added J10: DC Motor B, Connector_PinHeader_2.54mm:PinHeader_1x02_P2.54mm_Vertical, symbol Connector:Conn_01x02_Pin
- added J2: USB_C_Receptacle_USB2.0_16P, Connector_USB:USB_C_Receptacle_GCT_USB4105-xx-A_16P_TopMnt_Horizontal, symbol Connector:USB_C_Receptacle_USB2.0_16P
- added J3: VL53L0X_1, Connector_PinHeader_2.54mm:PinHeader_1x06_P2.54mm_Vertical, symbol Connector:Conn_01x06_Pin
- added J4: VL53L0X_2, Connector_PinHeader_2.54mm:PinHeader_1x06_P2.54mm_Vertical, symbol Connector:Conn_01x06_Pin
- added J5: Battery_connector, Connector_JST:JST_XH_B2B-XH-A_1x02_P2.50mm_Vertical, symbol Connector_Generic:Conn_01x02
- added J6: ELRS_Module, Connector_PinHeader_2.54mm:PinHeader_1x04_P2.54mm_Vertical, symbol Connector:Conn_01x04_Pin
- added J7: Tirette, Connector_JST:JST_XH_B2B-XH-A_1x02_P2.50mm_Vertical, symbol Connector_Generic:Conn_01x02
- added J8: DC Motor A, Connector_PinHeader_2.54mm:PinHeader_1x02_P2.54mm_Vertical, symbol Connector:Conn_01x02_Pin
- added J9: Odom_Shield, Connector_PinHeader_2.54mm:PinHeader_1x06_P2.54mm_Vertical, symbol Connector:Conn_01x06_Pin
- added Q1: PMOS, Package_TO_SOT_THT:TO-126-3_Vertical, symbol Simulation_SPICE:PMOS
- added R1, R2, R3, R5, R7, R8, R9: 10k, Resistor_SMD:R_1206_3216Metric, symbol Device:R
- added R4: 16.2k, Resistor_SMD:R_1206_3216Metric, symbol Device:R
- added R6: 1k, Resistor_SMD:R_1206_3216Metric, symbol Device:R
- added SW1, SW2: SW_Push, Button_Switch_SMD:SW_SPST_PTS810, symbol Switch:SW_Push
- added SW3: SW_Nidec_CAS-120A1, Button_Switch_SMD:Nidec_Copal_CAS-120A, symbol Switch:SW_Nidec_CAS-120A1
- added U2: USBLC6-2SC6, Package_TO_SOT_SMD:SOT-23-6, symbol Power_Protection:USBLC6-2SC6
- added U3: TLV76150DCY, Package_TO_SOT_SMD:SOT-223-3_TabPin2, symbol Regulator_Linear:TLV76150DCY
- added U4: TLV76133DCY, Package_TO_SOT_SMD:SOT-223-3_TabPin2, symbol Regulator_Linear:TLV76133DCY
- added U5: TB6612FNG, Custom_library:TB6612FNG_socket, symbol Custom_library:TB6612FNG
- U1: footprint ESP32-S3-WROOM-1U:ESP32-S3-WROOM-1U_EXP -> ESP32-S3-WROOM-1U_EXP
Connections:
- net GND: now reaches U1.1 (GND)
- net GND: now also U1.40 (GND), U1.41 (GND), U1.42 (GND), U1.43 (GND), U1.44 (GND), U1.45 (GND), U1.46 (GND), U1.47 (GND), U1.48 (GND), U1.49 (GND), C1.2, C10.2, C2.1, C3.1, C4.2, C5.1, C6.1, C7.1, C8.2, C9.2, D3.1 (K), J2.A1 (GND), J2.A12 (GND), J2.B1 (GND), J2.B12 (GND), J3.2 (GND), J4.2 (GND), J5.1 (Pin_1), J6.1 (GND), J9.1 (GND), Q1.2 (G), R1.1, R3.1, R5.1, SW1.1, SW2.1, SW3.1 (C), U2.2 (GND), U3.1 (GND), U4.1 (GND), U5.16 (GND), U5.3 (GND), U5.8 (GND)
- net ODOM_SCL: now reaches U1.10 (IO17)
- net ODOM_SCL: now also J9.4 (SCL)
- net ODOM_SDA: now reaches U1.11 (IO18)
- net ODOM_SDA: now also J9.3 (SDA)
- net TOF_SDA_1: now reaches U1.12 (IO8)
- net TOF_SDA_1: now also J3.3 (SCL), J4.3 (SCL)
- net D-: now reaches U1.13 (IO19_D-)
- net D-: now also U2.6 (I/O1)
- net D+: now reaches U1.14 (IO20_D+)
- net D+: now also U2.4 (I/O2)
- net TOF_SCL_1: now reaches U1.17 (IO9)
- net TOF_SCL_1: now also J3.4 (SDA), J4.4 (SDA)
- net PWMA: now reaches U1.18 (IO10)
- net PWMA: now also U5.9 (PWMA)
- net AIN1: now reaches U1.19 (IO11)
- net AIN1: now also U5.11 (AIN1)
- net +3.3V: now reaches U1.2 (3V3)
- net +3.3V: now also C1.1, C10.1, C4.1, J3.1 (VCC), J4.1 (VCC), J7.1 (Pin_1), J9.2 (3V3), R2.1, R7.1, R8.1, SW3.3 (A), U4.2 (VO), U5.2 (VCC)
- net AIN2: now reaches U1.20 (IO12)
- net AIN2: now also U5.10 (AIN2)
- net PWMB: now reaches U1.21 (IO13)
- net PWMB: now also U5.15 (PWMB)
- net BIN1: now reaches U1.22 (IO14)
- net BIN1: now also U5.13 (BIN1)
- net BIN2: now reaches U1.23 (IO21)
- net BIN2: now also U5.14 (BIN2)
- net STBY: now reaches U1.24 (IO47)
- net STBY: now also U5.12 (STBY)
- net BOOT: now reaches U1.27 (IO0)
- net BOOT: now also C3.2, SW2.2
- net EN: now reaches U1.3 (EN)
- net EN: now also C2.2, C5.2, R2.2, SW1.2
- net VBAT_SENSE: now reaches U1.31 (IO38)
- net VBAT_SENSE: now also R4.1, R5.2
- net ELRS_TX: now reaches U1.38 (IO2)
- net ELRS_TX: now also J6.3 (TX)
- net ELRS_RX: now reaches U1.39 (IO1)
- net ELRS_RX: now also J6.4 (RX)
- net TOF_SHUT_1: now reaches U1.4 (IO4)
- net TOF_SHUT_1: now also J3.6 (SHUT)
- net TOF_SHUT_2: now reaches U1.5 (IO5)
- net TOF_SHUT_2: now also J4.6 (SHUT)
- net TOF_INT_1: now reaches U1.6 (IO6)
- net TOF_INT_1: now also J3.5 (INT), R7.2
- net TOF_INT_2: now reaches U1.7 (IO7)
- net TOF_INT_2: now also J4.5 (INT), R8.2
- net MATCH_DIR: now reaches U1.8 (IO15)
- net MATCH_DIR: now also R9.1
- net TRIGGER: now reaches U1.9 (IO16)
- net TRIGGER: now also J7.2 (Pin_2)
- new net: J2.B5 (CC2), R1.2
- new net: D1.2 (A), J2.A4 (VBUS), J2.A9 (VBUS), J2.B4 (VBUS), J2.B9 (VBUS)
- new net: J2.A5 (CC1), R3.2
- new net: J2.A6 (D+), J2.B6 (D+), U2.3 (I/O2)
- new net: J2.A7 (D-), J2.B7 (D-), U2.1 (I/O1)
- new net: R9.2, SW3.2 (B)
- new net: D3.2 (A), R6.1
- new net: U3.2 (VO), U4.3 (VI)
- new net: J1.2 (Pin_2), Q1.1 (D)
- new net +5V: C9.1, J6.2 (5V)
- new net AO1: J8.1 (AO1), U5.4 (AO1)
- new net AO2: J8.2 (AO2), U5.5 (AO2)
- new net BAT_IN: J1.1 (Pin_1), J5.2 (Pin_2)
- new net BO1: J10.1 (BO1), U5.7 (BO1)
- new net BO2: J10.2 (BO2), U5.6 (BO2)
- new net VBAT: D2.2 (A), Q1.3 (S), R4.2, U5.1 (VM)
- new net VBUS: C6.2, C7.2, C8.1, D1.1 (K), D2.1 (K), R6.2, U2.5 (VBUS), U3.3 (VI)
- no-connect marks 0 -> 11
Other:
- note added: "3.3V Regulator"
- note added: "5V Regulator"
- note added: "Battery connector"
- note added: "DC Motors + driver"
- note added: "ELRS module"
- note added: "MCU + Reset/BOOT BTNs"
- note added: "Odometry Shield"
- note added: "PMOS should be able to tolerate 5A of current."
- note added: "Possible to unlock IOs 35-37 by using a chip with no PSRAM"
- note added: "Power Management"
- note added: "Schottky can be removed if the PMOS Vt is around 5V-6V and max Vsd is higher than 13V (USB plugged in and battery plugged in reverse)"
- note added: "TOF modules"
- note added: "Trigger pull + Direction selector"
- note added: "USB C port"
- note added: "Use internal pull-down"
- note added: "https://passionelectronique.fr/tutoriel-tb6612fng/"
- note added: "https://passionelectronique.fr/tutoriel-vl53l0x-arduino/"
- moved on the sheet: U1

Commit message: V1.1 : first layout
Parts:
- removed C8: 1uF, Capacitor_SMD:C_0805_2012Metric, symbol Device:C
- removed C9: 2.2uF, Capacitor_SMD:C_0805_2012Metric, symbol Device:C
- removed J10: DC Motor B, Connector_PinHeader_2.54mm:PinHeader_1x02_P2.54mm_Vertical, symbol Connector:Conn_01x02_Pin
- removed J8: DC Motor A, Connector_PinHeader_2.54mm:PinHeader_1x02_P2.54mm_Vertical, symbol Connector:Conn_01x02_Pin
- removed R9: 10k, Resistor_SMD:R_1206_3216Metric, symbol Device:R
- removed U3: TLV76150DCY, Package_TO_SOT_SMD:SOT-223-3_TabPin2, symbol Regulator_Linear:TLV76150DCY
- added C1, C5: 10uF, Capacitor_SMD:C_0805_2012Metric, symbol Device:C
- added C10: 0.1uF, Capacitor_SMD:C_0805_2012Metric, symbol Device:C
- added C11, C12: 22uF, Capacitor_SMD:C_0805_2012Metric, symbol Device:C
- added C13: 1uF, Capacitor_SMD:C_0805_2012Metric, symbol Device:C
- added H1, H2, H3, H4: MountingHole, MountingHole:MountingHole_2.2mm_M2, symbol Mechanical:MountingHole
- added J11: Conn_01x08_Pin, Connector_PinHeader_2.54mm:PinHeader_1x08_P2.54mm_Vertical, symbol Connector:Conn_01x08_Pin
- added J12: JTAG interface, Connector_PinHeader_2.54mm:PinHeader_1x04_P2.54mm_Vertical, symbol Connector:Conn_01x04_Pin
- added J7: DC Motor B, Connector_PinHeader_2.54mm:PinHeader_1x06_P2.54mm_Vertical, symbol Connector:Conn_01x06_Pin
- added J8: DC Motor A, Connector_PinHeader_2.54mm:PinHeader_1x06_P2.54mm_Vertical, symbol Connector:Conn_01x06_Pin
- added L1: 3.3uH, Inductor_SMD:L_0805_2012Metric, symbol Device:L
- added R5, R8: 10k, Resistor_SMD:R_1206_3216Metric, symbol Device:R
- added R7: 54k9, Resistor_SMD:R_1206_3216Metric, symbol Device:R
- added SW1: SW_Nidec_CAS-120A1, Button_Switch_SMD:Nidec_Copal_CAS-120A, symbol Switch:SW_Nidec_CAS-120A1
- added U1: TPS563201, Package_TO_SOT_SMD:SOT-23-6, symbol Regulator_Switching:TPS563201
- J1: value Emergency BTN -> Battery_connector
- R10: renamed from R6; value 1k -> 300
- R11: renamed from R8; now not fitted; now left out of the parts list
- R3: renamed from R1; value 10k -> 5k1
- R4: renamed from R3; value 10k -> 5k1
- R9: renamed from R7; now not fitted; now left out of the parts list
- renumbered C10 to C14, C1 to C2, C2 to C3, C3 to C4, C4 to C6, C6 to C7, C7 to C8, C5 to C9, D1 to D3, D3 to D4, J5 to J10, J7 to J5, R5 to R1, R4 to R2, R2 to R6, SW1 to SW2, SW2 to SW3, SW3 to SW4, U1 to U3
Connections:
- net +3.3V: now also J7.4 (VCC), J8.4 (VCC)
- net +5V: now also D3.2 (A), C11.1, C12.1, J11.1 (Pin_1), L1.2, R7.2
- net AIN2: now also U3.18 (IO10); no longer U3.20 (IO12)
- net AO1: now also J8.5 (MOT_+)
- net AO2: now also J8.6 (MOT_-)
- net BIN1: now also U3.21 (IO13); no longer U3.22 (IO14)
- net BIN2: now also U3.22 (IO14); no longer U3.23 (IO21)
- net BO1: now also J7.5 (MOT_+)
- net BO2: now also J7.6 (MOT_-)
- net ELRS_RX: now also U3.37 (IO43_TXD0); no longer U3.39 (IO1)
- net ELRS_TX: now also U3.36 (IO44_RXD0); no longer U3.38 (IO2)
- net GND: now also R1.2, C1.2, C11.2, C12.2, C13.2, C5.2, J11.2 (Pin_2), J11.3 (Pin_3), J7.1 (GND), J8.1 (GND), R8.2, SW1.3 (A), U1.1 (GND); no longer R1.1
- net MATCH_DIR: now also SW4.2 (B), U3.25 (IO48); no longer U3.8 (IO15)
- net ODOM_SCL: now also J3.4 (SDA), J4.4 (SDA), U3.38 (IO2); no longer U3.10 (IO17)
- net ODOM_SDA: now also J3.3 (SCL), J4.3 (SCL), U3.39 (IO1); no longer U3.11 (IO18)
- net PWMA: now also U3.17 (IO9); no longer U3.18 (IO10)
- net PWMB: now also U3.23 (IO21); no longer U3.21 (IO13)
- net STBY: now also U3.20 (IO12); no longer U3.24 (IO47)
- net TOF_INT_1: now also U3.29 (IO36); no longer U3.6 (IO6)
- net TOF_INT_2: now also U3.31 (IO38); no longer U3.7 (IO7)
- net TOF_SHUT_1: now also U3.28 (IO35); no longer U3.4 (IO4)
- net TOF_SHUT_2: now also U3.30 (IO37); no longer U3.5 (IO5)
- net TRIGGER: now also U3.24 (IO47); no longer U3.9 (IO16)
- net VBAT: now also C1.1, C5.1, R5.2, U1.3 (VIN); no longer D2.2 (A)
- net VBAT_SENSE: now also R1.1, U3.15 (IO3); no longer R1.2, U3.31 (IO38)
- net VBUS: now also D2.2 (A), J2.A4 (VBUS), J2.A9 (VBUS), J2.B4 (VBUS), J2.B9 (VBUS); no longer D2.1 (K), D3.1 (K), R10.2
- net TCK: now reaches U3.32 (IO39_MTCK)
- net TCK: now also J12.1 (TCK)
- net TDO: now reaches U3.33 (IO40_MTD0)
- net TDO: now also J12.2 (TDO)
- net TDI: now reaches U3.34 (IO41_MTDI)
- net TDI: now also J12.3 (TDI)
- net TMS: now reaches U3.35 (IO42_MTMS)
- net TMS: now also J12.4 (TMS)
- net USB_D+: now reaches J2.A6 (D+), J2.B6 (D+), U2.3 (I/O2)
- net USB_D-: now reaches J2.A7 (D-), J2.B7 (D-), U2.1 (I/O1)
- net at U4.3 (VI): now also D2.1 (K), D3.1 (K), R10.2, C13.1
- net at Q1.1 (D): now also SW1.2 (B); no longer J1.2 (Pin_2)
- removed net TOF_SCL_1: J3.4 (SDA), J4.4 (SDA), U3.17 (IO9)
- removed net TOF_SDA_1: J3.3 (SCL), J4.3 (SCL), U3.12 (IO8)
- new net: C10.1, L1.1, U1.2 (SW)
- new net: R7.1, R8.1, U1.4 (VFB)
- new net: R5.1, U1.5 (EN)
- new net: C10.2, U1.6 (VBST)
- new net: J1.2 (Pin_2), SW1.1 (C)
- new net ENC_AO1: J8.2 (ENC_1), U3.5 (IO5)
- new net ENC_AO2: J8.3 (ENC_2), U3.4 (IO4)
- new net ENC_BO1: J7.2 (ENC_1), U3.7 (IO7)
- new net ENC_BO2: J7.3 (ENC_2), U3.6 (IO6)
- new net IO15: J11.8 (Pin_8), U3.8 (IO15)
- new net IO16: J11.7 (Pin_7), U3.9 (IO16)
- new net IO17: J11.6 (Pin_6), U3.10 (IO17)
- new net IO18: J11.5 (Pin_5), U3.11 (IO18)
- new net IO8: J11.4 (Pin_4), U3.12 (IO8)
- no-connect marks 11 -> 7
Other:
- note added: "5V 3A Buck Regulator"
- note added: "Check if interrupt pin already has internal pull-up"
- note added: "JTAG interface"
- note added: "Make sure I²C devices each have a different address on the bus."
- note added: "Make sure the encoders are either push-pull or open-drain"
- note added: "Make sure to activate CDC in the IDE to disable default UART0 mapping for IOs 43 and 44"
- note added: "Mounting holes"
- note added: "PMOS should be able to tolerate 5A of current. (The physical switch as well)"
- note added: "Possible to use strapping pin IO3 if default state is not changed during boot period."
- note added: "Schottky can be removed if the PMOS max Vsd is higher than 8.4V (fully charged battery plugged in reverse)"
- note added: "Shield Actuators"
- note removed: "5V Regulator"
- note removed: "PMOS should be able to tolerate 5A of current."
- note removed: "Schottky can be removed if the PMOS Vt is around 5V-6V and max Vsd is higher than 13V (USB plugged in and battery plugged in reverse)"
- moved on the sheet: C14, C2, C3, C4, C6, C7, C8, C9, D3, D4, J10, J2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
